Commit message: Fix package structure: rename config, update setup.py, CMakeLists.txt, xacro, launch files, and imports
Co-authored-by: msirobot <148898439+msirobot@users.noreply.github.com>

File: multi_robot_simulation/urdf/diff_drive_robot.xacro (robot description, xacro)
@@ -1,6 +1,10 @@
 <?xml version="1.0"?>
-<robot name="diff_drive_robot" xmlns:xacro="http://www.ros.org/wiki/xacro">
+<robot xmlns:xacro="http://www.ros.org/wiki/xacro">
+  <!-- Define robot_name argument -->
+  <xacro:arg name="robot_name" default="robot"/>
+  <xacro:property name="robot_name" value="$(arg robot_name)"/>
+  <!-- Define the robot macro -->
   <xacro:macro name="diff_drive_robot" params="robot_name">
-    <link name="base_link">
+    <link name="${robot_name}/base_link">
       <visual>
         <geometry>
@@ -32,10 +36,19 @@
         <odometryTopic>odom</odometryTopic>
         <odometryFrame>odom</odometryFrame>
-        <robotBaseFrame>base_link</robotBaseFrame>
+        <robotBaseFrame>${robot_name}/base_link</robotBaseFrame>
+        <leftJoint>left_wheel_joint</leftJoint>
+        <rightJoint>right_wheel_joint</rightJoint>
+        <wheelSeparation>0.4</wheelSeparation>
+        <wheelDiameter>0.1</wheelDiameter>
+        <updateRate>10.0</updateRate>
+        <publishWheelTF>false</publishWheelTF>
+        <publishWheelJointState>false</publishWheelJointState>
       </plugin>
     </gazebo>
-    <gazebo reference="base_link">
+    <gazebo reference="${robot_name}/base_link">
       <material>Gazebo/Blue</material>
     </gazebo>
   </xacro:macro>
+  <!-- Instantiate the robot macro -->
+  <xacro:diff_drive_robot robot_name="${robot_name}"/>
 </robot>

Commit message: Add complete robot model with wheels and update README with usage instructions
Co-authored-by: msirobot <148898439+msirobot@users.noreply.github.com>

File: multi_robot_simulation/urdf/diff_drive_robot.xacro (robot description, xacro)
@@ -6,4 +6,5 @@
   <!-- Define the robot macro -->
   <xacro:macro name="diff_drive_robot" params="robot_name">
+    <!-- Base Link -->
     <link name="${robot_name}/base_link">
       <visual>
@@ -21,31 +22,129 @@
       </collision>
       <inertial>
-        <mass value="1.0"/>
-        <inertia ixx="0.01" ixy="0.0" ixz="0.0" iyy="0.01" iyz="0.0" izz="0.01"/>
+        <mass value="5.0"/>
+        <inertia ixx="0.1" ixy="0.0" ixz="0.0" iyy="0.1" iyz="0.0" izz="0.1"/>
       </inertial>
     </link>
-    <gazebo>
-      <plugin name="gazebo_ros_control" filename="libgazebo_ros_control.so">
-        <robotNamespace>/${robot_name}</robotNamespace>
-      </plugin>
-    </gazebo>
+    <!-- Left Wheel -->
+    <link name="${robot_name}/left_wheel">
+      <visual>
+        <geometry>
+          <cylinder length="0.05" radius="0.05"/>
+        </geometry>
+        <material name="black">
+          <color rgba="0 0 0 1"/>
+        </material>
+        <origin xyz="0 0 0" rpy="1.5707 0 0"/>
+      </visual>
+      <collision>
+        <geometry>
+          <cylinder length="0.05" radius="0.05"/>
+        </geometry>
+        <origin xyz="0 0 0" rpy="1.5707 0 0"/>
+      </collision>
+      <inertial>
+        <mass value="0.5"/>
+        <inertia ixx="0.001" ixy="0.0" ixz="0.0" iyy="0.001" iyz="0.0" izz="0.001"/>
+      </inertial>
+    </link>
+    <joint name="${robot_name}/left_wheel_joint" type="continuous">
+      <parent link="${robot_name}/base_link"/>
+      <child link="${robot_name}/left_wheel"/>
+      <origin xyz="0 0.225 0" rpy="0 0 0"/>
+      <axis xyz="0 1 0"/>
+    </joint>
+    <!-- Right Wheel -->
+    <link name="${robot_name}/right_wheel">
+      <visual>
+        <geometry>
+          <cylinder length="0.05" radius="0.05"/>
+        </geometry>
+        <material name="black">
+          <color rgba="0 0 0 1"/>
+        </material>
+        <origin xyz="0 0 0" rpy="1.5707 0 0"/>
+      </visual>
+      <collision>
+        <geometry>
+          <cylinder length="0.05" radius="0.05"/>
+        </geometry>
+        <origin xyz="0 0 0" rpy="1.5707 0 0"/>
+      </collision>
+      <inertial>
+        <mass value="0.5"/>
+        <inertia ixx="0.001" ixy="0.0" ixz="0.0" iyy="0.001" iyz="0.0" izz="0.001"/>
+      </inertial>
+    </link>
+    <joint name="${robot_name}/right_wheel_joint" type="continuous">
+      <parent link="${robot_name}/base_link"/>
+      <child link="${robot_name}/right_wheel"/>
+      <origin xyz="0 -0.225 0" rpy="0 0 0"/>
+      <axis xyz="0 1 0"/>
+    </joint>
+    <!-- Caster Wheel for stability -->
+    <link name="${robot_name}/caster_wheel">
+      <visual>
+        <geometry>
+          <sphere radius="0.025"/>
+        </geometry>
+        <material name="white">
+          <color rgba="1 1 1 1"/>
+        </material>
+      </visual>
+      <collision>
+        <geometry>
+          <sphere radius="0.025"/>
+        </geometry>
+      </collision>
+      <inertial>
+        <mass value="0.1"/>
+        <inertia ixx="0.0001" ixy="0.0" ixz="0.0" iyy="0.0001" iyz="0.0" izz="0.0001"/>
+      </inertial>
+    </link>
+    <joint name="${robot_name}/caster_wheel_joint" type="fixed">
+      <parent link="${robot_name}/base_link"/>
+      <child link="${robot_name}/caster_wheel"/>
+      <origin xyz="0.15 0 -0.075" rpy="0 0 0"/>
+    </joint>
+    <!-- Gazebo plugins -->
     <gazebo>
       <plugin name="diff_drive_controller" filename="libgazebo_ros_diff_drive.so">
         <robotNamespace>/${robot_name}</robotNamespace>
+        <alwaysOn>true</alwaysOn>
+        <updateRate>10.0</updateRate>
+        <leftJoint>${robot_name}/left_wheel_joint</leftJoint>
+        <rightJoint>${robot_name}/right_wheel_joint</rightJoint>
+        <wheelSeparation>0.45</wheelSeparation>
+        <wheelDiameter>0.1</wheelDiameter>
+        <wheelTorque>10</wheelTorque>
+        <wheelAcceleration>1.0</wheelAcceleration>
         <commandTopic>cmd_vel</commandTopic>
         <odometryTopic>odom</odometryTopic>
         <odometryFrame>odom</odometryFrame>
         <robotBaseFrame>${robot_name}/base_link</robotBaseFrame>
-        <leftJoint>left_wheel_joint</leftJoint>
-        <rightJoint>right_wheel_joint</rightJoint>
-        <wheelSeparation>0.4</wheelSeparation>
-        <wheelDiameter>0.1</wheelDiameter>
-        <updateRate>10.0</updateRate>
         <publishWheelTF>false</publishWheelTF>
+        <publishOdomTF>true</publishOdomTF>
         <publishWheelJointState>false</publishWheelJointState>
+        <legacyMode>false</legacyMode>
       </plugin>
     </gazebo>
+    <!-- Gazebo materials -->
     <gazebo reference="${robot_name}/base_link">
       <material>Gazebo/Blue</material>
+    </gazebo>
+    <gazebo reference="${robot_name}/left_wheel">
+      <material>Gazebo/Black</material>
+      <mu1>1.0</mu1>
+      <mu2>1.0</mu2>
+    </gazebo>
+    <gazebo reference="${robot_name}/right_wheel">
+      <material>Gazebo/Black</material>
+      <mu1>1.0</mu1>
+      <mu2>1.0</mu2>
+    </gazebo>
+    <gazebo reference="${robot_name}/caster_wheel">
+      <material>Gazebo/White</material>
+      <mu1>0.0</mu1>
+      <mu2>0.0</mu2>
     </gazebo>
   </xacro:macro>
